Commit message: Add custom locomotion changes: fast TD3 agent, new meshes, reward terms, remote control, and inference updates

File: src/holosoma/holosoma/data/robots/t1/t1_29dof.urdf (robot description, URDF)
Before this commit: robot T1, 32 links, 31 joints
Links:
- link left_hand_link: geometry collision cylinder length=0.15 radius=0.06; visual mesh filename=meshes/xinan.stl
- link right_hand_link: geometry collision cylinder length=0.15 radius=0.06; visual mesh filename=meshes/hanzo.stl
